File: probe/eagle/cheapboard1.0.brd (EAGLE design)
At the start: 106.7 x 34.3 mm, 9 parts, among them T1 BC547, U1 ATMEGA48A-AU

Commit message: Added many many new PCB files
Other:
- board size 106.7 x 34.3 mm -> 102.9 x 34.3 mm
Changed lines of the file:
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@@
 <setting verticaltext="up"/>
 </settings>
-<grid distance="0.005" unitdist="inch" unit="inch" style="lines" multiple="1" display="no" altdistance="0.025" altunitdist="inch" altunit="inch"/>
+<grid distance="0.05" unitdist="inch" unit="inch" style="lines" multiple="1" display="no" altdistance="0.025" altunitdist="inch" altunit="inch"/>
 <layers>
 <layer number="1" name="Top" color="4" fill="1" visible="yes" active="yes"/>
@@
 <wire x1="102.87" y1="0" x2="78.74" y2="11.43" width="0.4064" layer="20"/>
 <wire x1="78.74" y1="11.43" x2="68.58" y2="11.43" width="0.4064" layer="20"/>
-<wire x1="68.58" y1="11.43" x2="68.58" y2="13.97" width="0.4064" layer="20"/>
-<wire x1="68.58" y1="13.97" x2="97.79" y2="13.97" width="0.4064" layer="20"/>
-<wire x1="97.79" y1="13.97" x2="106.68" y2="17.78" width="0.4064" layer="20"/>
-<wire x1="106.68" y1="17.78" x2="97.79" y2="20.32" width="0.4064" layer="20"/>
-<wire x1="97.79" y1="20.32" x2="68.58" y2="20.32" width="0.4064" layer="20"/>
-<wire x1="68.58" y1="20.32" x2="68.58" y2="22.86" width="0.4064" layer="20"/>
+<wire x1="68.58" y1="11.43" x2="68.58" y2="22.86" width="0.4064" layer="20"/>
 <wire x1="68.58" y1="22.86" x2="80.01" y2="22.86" width="0.4064" layer="20"/>
 <wire x1="80.01" y1="22.86" x2="102.87" y2="34.29" width="0.4064" layer="20"/>
