File: probe/eagle/cheapboard1.1.brd (EAGLE design)
At the start: 105.4 x 34.3 mm, 20 parts, among them J1 AVR_SPI_PRG_6OFFSET_PADS, T1 BC547, U2 ATMEGA8U2-MU

Commit message: Added final design for v1.1 manufacture
Parts:
- added LED1, LED2, LED3, LED4, LED5: (no value), led:CHIPLED_0805
- added R10, R11, R12, R13, R8, R9: (no value), rcl:M0805
- added S1, S2: (no value), SparkFun-Electromechanical:TACTILE_SWITCH_SMD
- moved R3 2.67 mm to (50.4, 17.4)
Connections:
- new net N$19: LED1.A, U2.5
- new net N$20: LED2.A, U2.26
- new net N$21: LED3.A, U2.25
- new net N$22: LED4.A, U2.23
- new net N$23: LED5.A, U2.22
- new net N$24: LED1.C, R8.2
- new net N$25: LED2.C, R9.2
- new net N$26: LED3.C, R10.2
- new net N$27: LED4.C, R11.2
- new net N$28: LED5.C, R12.2
- new net N$30: R13.2, S2.1, S2.2, U2.11
- net GND: now also R10.1, R11.1, R12.1, R13.1, R8.1, R9.1, S1.1
- net N$4: now also S1.3, S1.4
- net VCC: now also S2.3, S2.4
Routing:
- net GND: track 138.5 -> 247.6 mm, vias 0 -> 3
- net VCC: track 5.53 -> 46.1 mm, vias 0 -> 2
- net N$30: track 0.00 -> 32.9 mm, vias 0 -> 1
- net N$22: track 0.00 -> 28.8 mm, vias 0 -> 1
- net N$23: track 0.00 -> 19.0 mm, vias 0 -> 1
- net N$19: track 0.00 -> 18.8 mm, vias 0 -> 1
- net N$21: track 0.00 -> 18.1 mm, vias 0 -> 1
- net N$9: track 5.62 -> 22.4 mm, vias 0 -> 2
- net N$20: track 0.00 -> 15.7 mm, vias 0 -> 1
- net N$4: track 35.4 -> 45.6 mm
- net N$14: track 83.1 -> 85.7 mm
- net N$18: track 10.3 -> 8.04 mm
- net N$25: track 0.00 -> 2.18 mm
- net N$26: track 0.00 -> 2.17 mm
- net N$28: track 0.00 -> 2.16 mm
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Other:
- board text added: "Ben Oxley"
- board text added: "Soil Lite V1.1"
