File: probe/eagle/cheapboard1.1qfn.sch (EAGLE design)
At the start: 33 parts, among them J1 AVR_SPI_PRG_6OFFSET_PADS, T1 BC547, U2 ATMEGA8U2-MU

Commit message: Added final design for v1.1 manufacture
Parts:
- added C5, C6: (no value), SparkFun-Passives:CAP0805
- added JP2: FTDI_DEVICE, SparkFun-Connectors:FTDI_DEVICE
- added R14, R15, R16: (no value), rcl:R-EU_M0805
- added U1: AT25256B-SSHL-B, Mine:AT25256B-SSHL-B
- BAT1: device special:BATTERY -> SparkFun-Electromechanical:BATTERY245PTH
- T1: value BC547 -> (none); device transistor:BC547 -> SparkFun-DiscreteSemi:TRANSISTOR_NPNSOT23-3
- Y1: value (none) -> 8MHz
Connections:
- new net DTR: JP2.DTR, U2.PD7
- new net N$29: R15.1, U1.SI
- new net N$31: R16.2, U1.SO
- new net N$34: U1.~CS, U2.PB4
- new net N$35: U1.~WP, U2.PB7
- new net N$36: U1.~HOLD, U2.PB5
- new net RX: JP2.TXO, U2.PD2
- new net TX: JP2.RXI, U2.PD3
- net GND: now also C5.2, C6.2, JP1.GND, JP2.CTS, JP2.GND, U1.GND, U2.EP, U2.UGND
- net N$1: now also U2.PD0; no longer U2.PD3
- net N$10: now also U2.D-; no longer U2.D+
- net N$11: now also U2.D+; no longer U2.D-
- net N$14: now also U2.PD1; no longer U2.PD7
- net N$15: now also R14.1, U1.SCK; no longer JP1.GND, U2.UGND
- net N$2: now also R15.2
- net N$5: now also R14.2
- net N$7: now also R16.1
- net VCC: now also C5.1, C6.1, JP2.VCC, U1.VCC
Other:
- moved on the sheet: C2, R4, R5
